Commit message: Made vpython visualization for robot arm from URDF, angle changes are HEAVILY HARDCODED

File: PingPongRobot/arm_urdf.urdf (robot description, URDF)
Before this commit: robot robot_arm, 6 links, 5 joints
Joints:
- joint base_joint: origin xyz=0 0 0 rpy=0 0 0 -> xyz=0 0 0.0375 rpy=0 0 0
- joint elbow_joint: origin xyz=0 0 0.28 rpy=0 0 0 -> xyz=-0.07 0 0.28 rpy=0 0 0
- joint shoulder_joint: origin xyz=0 0 0.06 rpy=0 0 0 -> xyz=0.1 0 0.0225 rpy=0 0 0
- joint wrist_joint: origin xyz=0 0 0.28 rpy=0 0 0 -> xyz=0.07 0 0.28 rpy=0 0 0
- joint wrist_rotor_joint: origin xyz=0.1 0 0.21 rpy=0 0 0 -> xyz=0 0 0.21 rpy=0 0 0

Commit message: added ik to the simulated vpython arm, tested accuracy and rotations etc

File: PingPongRobot/arm_urdf.urdf (robot description, URDF)
Before this commit: robot robot_arm, 6 links, 5 joints
Joints:
- joint base_joint: limit lower=-3.14159 upper=3.14159 -> lower=-50 upper=50
- joint elbow_joint: limit lower=-2 upper=2 -> lower=-2.5 upper=2.5
- joint shoulder_joint: limit lower=-1.2 upper=1.2 -> lower=-1.57 upper=1.57

Commit message: some extra stuff, and created new integration file

File: PingPongRobot/arm_urdf.urdf (robot description, URDF)
Before this commit: robot robot_arm, 6 links, 5 joints
Links:
- added link handle; visual box size=0.03 0.02 0.1
- added link paddle; visual box size=0.15 0.02 0.2
- added link paddle_center
Joints:
- added joint end_effector: type fixed, parent paddle, child paddle_center, origin xyz=0 0 0.1 rpy=0 0 0
- added joint handle_paddle_joint: type fixed, parent handle, child paddle, origin xyz=0 0 0.1 rpy=0 0 0
- added joint wrist_handle_joint: type fixed, parent wrist_rotor, child handle, origin xyz=0 0 0 rpy=0 0 0
